File: schematic/kicad/f1_car/f1_car.kicad_pcb (KiCad board)
At the start: 2 copper layers, 27.9 x 62.4 mm, 2 parts, among them J4 Conn_01x12_Pin, U1 ESP32-C3-DevKitC-02

Commit message: added b silkscreen
Other:
- board text added: "PFI E-Racing"
Changed lines of the file:
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@@
   (gr_line (start 133.27654 129.826) (end 158.160036 129.826)
     (stroke (width 0.05) (type default)) (layer "Edge.Cuts"))
+  (gr_text "PFI E-Racing" (at 146.745104 88.292351 90) (layer "B.SilkS")
+    (effects (font (size 2 2) (thickness 0.15)) (justify left bottom mirror))
+  )
   (gr_text "+5V" (at 135.4 83.45 90) (layer "F.SilkS")
     (effects (font (size 1 1) (thickness 0.15)) (justify left bottom))
