File: schematic/kicad/f1_car/f1_car.kicad_sch (KiCad schematic)
At the start: 5 parts, among them J4 Conn_01x12_Pin, U1 ESP32-C3-DevKitC-02

Commit message: jlcpcb design rules constraints
Other:
- moved on the sheet: J1, J2, J3, J4
